Commit message: fix: add dummy root link

File: src/ros2/nxt_rover/urdf/simple_rover.urdf.xacro (robot description, xacro)
@@ -12,4 +12,11 @@
   <xacro:property name="caster_radius" value="0.03"/>
   <xacro:property name="caster_mass" value="0.1"/>
+  <!-- Dummy root link to avoid KDL root-inertia warning -->
+  <link name="base_link_root"/>
+  <joint name="root_to_base_link" type="fixed">
+    <parent link="base_link_root"/>
+    <child link="base_link"/>
+    <origin xyz="0 0 0" rpy="0 0 0"/>
+  </joint>
   <!-- Base link -->
   <link name="base_link">

Commit message: feat: xacro experiments

File: src/ros2/nxt_rover/urdf/simple_rover.urdf.xacro (robot description, xacro)
@@ -1,16 +1,17 @@
 <?xml version="1.0"?>
 <robot name="simple_rover" xmlns:xacro="http://www.ros.org/wiki/xacro">
-  <!-- Simple differential-drive rover: base + two drive wheels + rear caster -->
+  <!-- Simple 4-wheel rover: front steering + four wheels -->
   <!-- Parameters -->
-  <xacro:property name="wheel_radius" value="0.06"/>
-  <xacro:property name="wheel_width" value="0.02"/>
-  <xacro:property name="base_length" value="0.4"/>
-  <xacro:property name="base_width" value="0.28"/>
-  <xacro:property name="base_height" value="0.08"/>
-  <xacro:property name="base_mass" value="5.0"/>
-  <xacro:property name="wheel_mass" value="0.5"/>
-  <xacro:property name="caster_radius" value="0.03"/>
-  <xacro:property name="caster_mass" value="0.1"/>
-  <!-- Dummy root link to avoid KDL root-inertia warning -->
+  <xacro:property name="wheel_radius" value="0.08"/>
+  <xacro:property name="wheel_width" value="0.04"/>
+  <xacro:property name="wheel_base" value="0.35"/> <!-- distance between front and rear axles -->
+  <xacro:property name="track_width" value="0.22"/> <!-- distance between left and right wheels -->
+  <xacro:property name="chassis_length" value="${wheel_base + 0.15}"/>
+  <xacro:property name="chassis_width" value="${track_width + 0.06}"/>
+  <xacro:property name="chassis_height" value="0.12"/>
+  <xacro:property name="chassis_mass" value="12.0"/>
+  <xacro:property name="wheel_mass" value="1.0"/>
+  <xacro:property name="steer_mass" value="0.1"/>
+  <!-- Root link -->
   <link name="base_link_root"/>
   <joint name="root_to_base_link" type="fixed">
@@ -19,124 +20,189 @@
     <origin xyz="0 0 0" rpy="0 0 0"/>
   </joint>
-  <!-- Base link -->
+  <!-- Chassis -->
   <link name="base_link">
     <inertial>
-      <origin xyz="0 0 0" rpy="0 0 0"/>
-      <mass value="${base_mass}"/>
-      <!-- Approximate inertia for a rectangular box -->
-      <inertia ixx="${(1.0/12.0)*base_mass*(base_height*base_height + base_length*base_length)}"
+      <origin xyz="0 0 ${wheel_radius + chassis_height/2.0}" rpy="0 0 0"/>
+      <mass value="${chassis_mass}"/>
+      <!-- Simple box inertia approximation -->
+      <inertia ixx="${(1.0/12.0)*chassis_mass*(chassis_height*chassis_height + chassis_length*chassis_length)}"
                ixy="0" ixz="0"
-               iyy="${(1.0/12.0)*base_mass*(base_width*base_width + base_length*base_length)}" iyz="0"
-               izz="${(1.0/12.0)*base_mass*(base_width*base_width + base_height*base_height)}"/>
-    </inertial>
-    <visual>
-      <origin xyz="0 0 ${base_height/2.0}" rpy="0 0 0"/>
-      <geometry>
-        <box size="${base_length} ${base_width} ${base_height}"/>
-      </geometry>
-      <material name="gray"><color rgba="0.6 0.6 0.6 1.0"/></material>
-    </visual>
-    <collision>
-      <origin xyz="0 0 ${base_height/2.0}" rpy="0 0 0"/>
-      <geometry>
-        <box size="${base_length} ${base_width} ${base_height}"/>
-      </geometry>
-    </collision>
-  </link>
-  <!-- Wheels -->
-  <!-- Positions: front-left, front-right (x forward, y left positive, z up) -->
-  <link name="left_wheel">
-    <inertial>
-      <origin xyz="0 0 0" rpy="0 0 0"/>
-      <mass value="${wheel_mass}"/>
-      <!-- cylinder approx inertia about center for axis = y -->
-      <inertia ixx="${0.5*wheel_mass*wheel_radius*wheel_radius}" ixy="0" ixz="0"
-               iyy="${(1.0/12.0)*wheel_mass*(2*wheel_radius*2*wheel_radius + wheel_width*wheel_width)}" iyz="0"
-               izz="${0.5*wheel_mass*wheel_radius*wheel_radius}"/>
-    </inertial>
-    <visual>
-      <origin xyz="0 0 0" rpy="0 0 0"/>
-      <geometry>
-        <cylinder length="${wheel_width}" radius="${wheel_radius}"/>
-      </geometry>
-      <material name="black"><color rgba="0 0 0 1.0"/></material>
-    </visual>
-    <collision>
-      <origin xyz="0 0 0" rpy="0 0 0"/>
-      <geometry>
-        <cylinder length="${wheel_width}" radius="${wheel_radius}"/>
-      </geometry>
-    </collision>
-  </link>
-  <link name="right_wheel">
-    <inertial>
-      <origin xyz="0 0 0" rpy="0 0 0"/>
-      <mass value="${wheel_mass}"/>
-      <inertia ixx="${0.5*wheel_mass*wheel_radius*wheel_radius}" ixy="0" ixz="0"
-               iyy="${(1.0/12.0)*wheel_mass*(2*wheel_radius*2*wheel_radius + wheel_width*wheel_width)}" iyz="0"
-               izz="${0.5*wheel_mass*wheel_radius*wheel_radius}"/>
-    </inertial>
-    <visual>
-      <origin xyz="0 0 0" rpy="0 0 0"/>
-      <geometry>
-        <cylinder length="${wheel_width}" radius="${wheel_radius}"/>
-      </geometry>
-      <material name="black"><color rgba="0 0 0 1.0"/></material>
-    </visual>
-    <collision>
-      <origin xyz="0 0 0" rpy="0 0 0"/>
-      <geometry>
-        <cylinder length="${wheel_width}" radius="${wheel_radius}"/>
-      </geometry>
-    </collision>
-  </link>
-  <!-- Rear caster (simple small wheel, fixed orientation) -->
-  <link name="caster_wheel">
-    <inertial>
-      <origin xyz="0 0 0" rpy="0 0 0"/>
-      <mass value="${caster_mass}"/>
+               iyy="${(1.0/12.0)*chassis_mass*(chassis_width*chassis_width + chassis_length*chassis_length)}" iyz="0"
+               izz="${(1.0/12.0)*chassis_mass*(chassis_width*chassis_width + chassis_height*chassis_height)}"/>
+    </inertial>
+    <visual>
+      <origin xyz="0 0 ${wheel_radius + chassis_height/2.0}" rpy="0 0 0"/>
+      <geometry>
+        <box size="${chassis_length} ${chassis_width} ${chassis_height}"/>
+      </geometry>
+      <material name="blue"><color rgba="0.2 0.4 0.8 1.0"/></material>
+    </visual>
+    <collision>
+      <origin xyz="0 0 ${wheel_radius + chassis_height/2.0}" rpy="0 0 0"/>
+      <geometry>
+        <box size="${chassis_length} ${chassis_width} ${chassis_height}"/>
+      </geometry>
+    </collision>
+  </link>
+  <!-- Steering links (small mass-less links to steer front wheels) -->
+  <link name="front_left_steer">
+    <inertial>
+      <origin xyz="0 0 0" rpy="0 0 0"/>
+      <mass value="${steer_mass}"/>
       <inertia ixx="0.0001" ixy="0" ixz="0" iyy="0.0001" iyz="0" izz="0.0001"/>
     </inertial>
-    <visual>
-      <origin xyz="0 0 0" rpy="0 0 0"/>
-      <geometry>
-        <sphere radius="${caster_radius}"/>
-      </geometry>
-      <material name="dark"><color rgba="0.2 0.2 0.2 1.0"/></material>
-    </visual>
-  </link>
-  <!-- Wheel joints -->
-  <!-- Wheel centers are placed near the lower edges of the base -->
-  <joint name="left_wheel_joint" type="continuous">
-    <parent link="base_link"/>
-    <child link="left_wheel"/>
-    <!-- place at left side, slightly forward -->
-    <origin xyz="${base_length*0.2} ${base_width/2.0 + wheel_width/2.0} ${wheel_radius}" rpy="0 0 0"/>
-    <!-- rotate about robot Y axis to spin the wheel -->
-    <axis xyz="0 1 0"/>
-  </joint>
-  <joint name="right_wheel_joint" type="continuous">
-    <parent link="base_link"/>
-    <child link="right_wheel"/>
-    <origin xyz="${base_length*0.2} ${-(base_width/2.0 + wheel_width/2.0)} ${wheel_radius}" rpy="0 0 0"/>
-    <axis xyz="0 1 0"/>
-  </joint>
-  <!-- Caster fixed to the rear center of base -->
-  <joint name="caster_joint" type="fixed">
-    <parent link="base_link"/>
-    <child link="caster_wheel"/>
-    <origin xyz="${-base_length*0.35} 0 ${caster_radius}" rpy="0 0 0"/>
-  </joint>
-  <!-- Basic sensors or frames to attach sensors to -->
+  </link>
+  <link name="front_right_steer">
+    <inertial>
+      <origin xyz="0 0 0" rpy="0 0 0"/>
+      <mass value="${steer_mass}"/>
+      <inertia ixx="0.0001" ixy="0" ixz="0" iyy="0.0001" iyz="0" izz="0.0001"/>
+    </inertial>
+  </link>
+  <!-- Wheel definitions -->
+  <link name="front_left_wheel">
+    <inertial>
+      <origin xyz="0 0 0" rpy="0 0 0"/>
+      <mass value="${wheel_mass}"/>
+      <inertia ixx="${0.5*wheel_mass*wheel_radius*wheel_radius}" ixy="0" ixz="0"
+               iyy="${(1.0/12.0)*wheel_mass*(2*wheel_radius*2*wheel_radius + wheel_width*wheel_width)}" iyz="0"
+               izz="${0.5*wheel_mass*wheel_radius*wheel_radius}"/>
+    </inertial>
+    <visual>
+      <origin xyz="0 0 0" rpy="0 0 0"/>
+      <geometry>
+        <cylinder length="${wheel_width}" radius="${wheel_radius}"/>
+      </geometry>
+      <material name="black"><color rgba="0 0 0 1"/></material>
+    </visual>
+    <collision>
+      <origin xyz="0 0 0" rpy="0 0 0"/>
+      <geometry>
+        <cylinder length="${wheel_width}" radius="${wheel_radius}"/>
+      </geometry>
+    </collision>
+  </link>
+  <link name="front_right_wheel">
+    <inertial>
+      <origin xyz="0 0 0" rpy="0 0 0"/>
+      <mass value="${wheel_mass}"/>
+      <inertia ixx="${0.5*wheel_mass*wheel_radius*wheel_radius}" ixy="0" ixz="0"
+               iyy="${(1.0/12.0)*wheel_mass*(2*wheel_radius*2*wheel_radius + wheel_width*wheel_width)}" iyz="0"
+               izz="${0.5*wheel_mass*wheel_radius*wheel_radius}"/>
+    </inertial>
+    <visual>
+      <origin xyz="0 0 0" rpy="0 0 0"/>
+      <geometry>
+        <cylinder length="${wheel_width}" radius="${wheel_radius}"/>
+      </geometry>
+      <material name="black"><color rgba="0 0 0 1"/></material>
+    </visual>
+    <collision>
+      <origin xyz="0 0 0" rpy="0 0 0"/>
+      <geometry>
+        <cylinder length="${wheel_width}" radius="${wheel_radius}"/>
+      </geometry>
+    </collision>
+  </link>
+  <link name="rear_left_wheel">
+    <inertial>
+      <origin xyz="0 0 0" rpy="0 0 0"/>
+      <mass value="${wheel_mass}"/>
+      <inertia ixx="${0.5*wheel_mass*wheel_radius*wheel_radius}" ixy="0" ixz="0"
+               iyy="${(1.0/12.0)*wheel_mass*(2*wheel_radius*2*wheel_radius + wheel_width*wheel_width)}" iyz="0"
+               izz="${0.5*wheel_mass*wheel_radius*wheel_radius}"/>
+    </inertial>
+    <visual>
+      <origin xyz="0 0 0" rpy="0 0 0"/>
+      <geometry>
+        <cylinder length="${wheel_width}" radius="${wheel_radius}"/>
+      </geometry>
+      <material name="black"><color rgba="0 0 0 1"/></material>
+    </visual>
+    <collision>
+      <origin xyz="0 0 0" rpy="0 0 0"/>
+      <geometry>
+        <cylinder length="${wheel_width}" radius="${wheel_radius}"/>
+      </geometry>
+    </collision>
+  </link>
+  <link name="rear_right_wheel">
+    <inertial>
+      <origin xyz="0 0 0" rpy="0 0 0"/>
+      <mass value="${wheel_mass}"/>
+      <inertia ixx="${0.5*wheel_mass*wheel_radius*wheel_radius}" ixy="0" ixz="0"
+               iyy="${(1.0/12.0)*wheel_mass*(2*wheel_radius*2*wheel_radius + wheel_width*wheel_width)}" iyz="0"
+               izz="${0.5*wheel_mass*wheel_radius*wheel_radius}"/>
+    </inertial>
+    <visual>
+      <origin xyz="0 0 0" rpy="0 0 0"/>
+      <geometry>
+        <cylinder length="${wheel_width}" radius="${wheel_radius}"/>
+      </geometry>
+      <material name="black"><color rgba="0 0 0 1"/></material>
+    </visual>
+    <collision>
+      <origin xyz="0 0 0" rpy="0 0 0"/>
+      <geometry>
+        <cylinder length="${wheel_width}" radius="${wheel_radius}"/>
+      </geometry>
+    </collision>
+  </link>
+  <!-- Joints -->
+  <!-- Front steering (yaw) joints -->
+  <joint name="front_left_steer_joint" type="revolute">
+    <parent link="base_link"/>
+    <child link="front_left_steer"/>
+    <origin xyz="${wheel_base/2.0} ${track_width/2.0} ${wheel_radius}" rpy="0 0 0"/>
+    <axis xyz="0 0 1"/>
+    <limit lower="-0.785" upper="0.785" effort="10" velocity="1.0"/>
+  </joint>
+  <joint name="front_right_steer_joint" type="revolute">
+    <parent link="base_link"/>
+    <child link="front_right_steer"/>
+    <origin xyz="${wheel_base/2.0} ${-track_width/2.0} ${wheel_radius}" rpy="0 0 0"/>
+    <axis xyz="0 0 1"/>
+    <limit lower="-0.785" upper="0.785" effort="10" velocity="1.0"/>
+  </joint>
+  <!-- Wheel spin joints (rotate around robot Y axis) -->
+  <joint name="front_left_wheel_joint" type="continuous">
+    <parent link="front_left_steer"/>
+    <child link="front_left_wheel"/>
+    <origin xyz="0 0 0" rpy="0 0 0"/>
+    <axis xyz="0 1 0"/>
+  </joint>
+  <joint name="front_right_wheel_joint" type="continuous">
+    <parent link="front_right_steer"/>
+    <child link="front_right_wheel"/>
+    <origin xyz="0 0 0" rpy="0 0 0"/>
+    <axis xyz="0 1 0"/>
+  </joint>
+  <joint name="rear_left_wheel_joint" type="continuous">
+    <parent link="base_link"/>
+    <child link="rear_left_wheel"/>
+    <origin xyz="${-wheel_base/2.0} ${track_width/2.0} ${wheel_radius}" rpy="0 0 0"/>
+    <axis xyz="0 1 0"/>
+  </joint>
+  <joint name="rear_right_wheel_joint" type="continuous">
+    <parent link="base_link"/>
+    <child link="rear_right_wheel"/>
+    <origin xyz="${-wheel_base/2.0} ${-track_width/2.0} ${wheel_radius}" rpy="0 0 0"/>
+    <axis xyz="0 1 0"/>
+  </joint>
+  <!-- IMU frame -->
   <link name="imu_link"/>
   <joint name="imu_joint" type="fixed">
     <parent link="base_link"/>
     <child link="imu_link"/>
-    <origin xyz="0 0 ${base_height + 0.02}" rpy="0 0 0"/>
-  </joint>
-  <!-- Simple tags to make simulation easy -->
-  <gazebo reference="left_wheel">
-    <mu1>0.0</mu1>
-    <mu2>0.0</mu2>
+    <origin xyz="0 0 ${wheel_radius + chassis_height}" rpy="0 0 0"/>
+  </joint>
+  <!-- Gazebo hints -->
+  <gazebo reference="front_left_wheel">
+    <mu1>0.8</mu1>
+    <mu2>0.8</mu2>
+  </gazebo>
+  <gazebo reference="front_right_wheel">
+    <mu1>0.8</mu1>
+    <mu2>0.8</mu2>
   </gazebo>
 </robot>
